Commit message: ros2 control and services commit

File: arduinobot_description/urdf/arduinobot.xacro (robot description, xacro)
@@ -6,4 +6,8 @@
     <xacro:property name="velocity" value="30.0"/>
     <xacro:property name="effort" value="10.0"/>
+    <!-- Gazebo plugin file-->
+    <xacro:include filename="$(find arduinobot_description)/urdf/arduinobot_gazebo.xacro"/>
+    <!-- ros2 control -->
+    <xacro:include filename="$(find arduinobot_description)/urdf/arduinobot_control.xacro"/>
 <!-- Inertial macro -->
 <xacro:macro name="default_inertial" params="mass">
@@ -14,5 +18,5 @@
 </xacro:macro>
 <!-- Transmission macro -->
-<xacro:macro name="default_transmisiion" params="joint">
+<xacro:macro name="default_transmission" params="joint">
     <transmission name="${joint}_transmission">
         <type>transmission_interface/SimpleTransmission</type>
@@ -175,5 +179,4 @@
     <parent link = "horizontal_arm"/>
     <child link = "claw_support"/>
-    <limit effort = "${effort}" lower = "-${PI/2}" upper = "${PI/2}" velocity = "${velocity}"/>
 </joint>
 <!-- Joint 5 (claw_support_to_right_gripper_finger)-->
@@ -195,7 +198,7 @@
 </joint>
 <!-- Transmissions -->
-<xacro:default_transmission params = "joint_1"/>
-<xacro:default_transmission params = "joint_2"/>
-<xacro:default_transmission params = "joint_3"/>
-<xacro:default_transmission params = "horizontal_arm_to_claw_support"/>
+<xacro:default_transmission joint = "joint_1"/>
+<xacro:default_transmission joint = "joint_2"/>
+<xacro:default_transmission joint = "joint_3"/>
+<xacro:default_transmission joint = "horizontal_arm_to_claw_support"/>
 </robot>

Commit message: made corrections on xacro file

File: arduinobot_description/urdf/arduinobot.xacro (robot description, xacro)
@@ -50,5 +50,5 @@
     <xacro:default_inertial mass = "0.1"/>
     <visual>
-        <origin xyz="-0.39 -0.39 -0.28" rpy="0.0 0.0 0.0"/>
+        <origin xyz="-0.39 -0.39 -0.56" rpy="0.0 0.0 0.0"/>
         <geometry>
             <mesh filename="package://arduinobot_description/meshes/base_plate.STL" scale="0.01 0.01 0.01"/>
@@ -56,5 +56,5 @@
     </visual>
     <collision>
-        <origin xyz="-0.39 -0.39 -0.28" rpy="0.0 0.0 0.0"/>
+        <origin xyz="-0.39 -0.39 -0.56" rpy="0.0 0.0 0.0"/>
         <geometry>
             <mesh filename="package://arduinobot_description/meshes/base_plate.STL" scale="0.01 0.01 0.01"/>
@@ -66,4 +66,5 @@
     <xacro:default_inertial mass = "0.1"/>
     <visual>
+        <!-- <origin xyz="0.19 0.06 0.28" rpy="0.0 -${PI/2} ${PI/2}"/> -->
         <origin xyz="0.19 0.06 -0.08" rpy="0.0 -${PI/2} ${PI/2}"/>
         <geometry>
@@ -146,13 +147,13 @@
 <!-- Virtual joint-->
 <joint name="virtual_joint" type="fixed">
-    <origin xyz="0.0 0.0 0.0" rpy="0.0 0.0 0.0"/>
     <parent link="world"/>
     <child link="base_link"/>
+    <origin xyz="0.0 0.0 0.0" />
 </joint>
 <!-- Joint 1-->
 <joint name="joint_1" type="revolute">
-    <origin xyz="0.0 0.0 0.0" rpy="0.0 0.0 0.0"/>
     <parent link="base_link"/>
     <child link="base_plate"/>
+    <origin xyz="0.0 0.0 0.307" rpy="0.0 0.0 0.0"/>
     <axis xyz="0.0 0.0 1.0"/>
     <limit effort="${effort}" lower="-${PI/2}" upper="${PI/2}" velocity="${velocity}"/>
@@ -160,5 +161,5 @@
 <!-- Joint 2-->
 <joint name = "joint_2" type="revolute">
-    <origin xyz = "-0.02 0.0 0.35" rpy = "0.0 0.0 0.0"/>
+    <origin xyz="-0.02 0 0.35"/>
     <parent link = "base_plate"/>
     <child link = "forward_drive_arm"/>

Commit message: added camera in the urdf

File: arduinobot_description/urdf/arduinobot.xacro (robot description, xacro)
@@ -6,25 +6,27 @@
     <xacro:property name="velocity" value="30.0"/>
     <xacro:property name="effort" value="10.0"/>
+    <!-- Inertial macro -->
+    <xacro:macro name="default_inertial" params="mass">
+        <inertial>
+            <mass value="${mass}"/>
+            <inertia ixx="1.0" ixy="0.0" ixz="0.0" iyy="1.0" iyz="0.0" izz="1.0"/>
+        </inertial>
+    </xacro:macro>
+    <!-- Transmission macro -->
+    <xacro:macro name="default_transmission" params="joint">
+        <transmission name="${joint}_transmission">
+            <type>transmission_interface/SimpleTransmission</type>
+            <joint name="${joint}" role = "joint_1">
+                <mechanicalReduction>1.0</mechanicalReduction>
+            </joint>
+            <actuator name="${joint}_motor" role = "actuator_1"/>
+        </transmission>
+    </xacro:macro>
+    <!-- Camera urdf-->
+    <xacro:include filename="$(find arduinobot_description)/urdf/arduinobot_camera.xacro"/>
     <!-- Gazebo plugin file-->
     <xacro:include filename="$(find arduinobot_description)/urdf/arduinobot_gazebo.xacro"/>
     <!-- ros2 control -->
     <xacro:include filename="$(find arduinobot_description)/urdf/arduinobot_control.xacro"/>
-<!-- Inertial macro -->
-<xacro:macro name="default_inertial" params="mass">
-    <inertial>
-        <mass value="${mass}"/>
-        <inertia ixx="1.0" ixy="0.0" ixz="0.0" iyy="1.0" iyz="0.0" izz="1.0"/>
-    </inertial>
-</xacro:macro>
-<!-- Transmission macro -->
-<xacro:macro name="default_transmission" params="joint">
-    <transmission name="${joint}_transmission">
-        <type>transmission_interface/SimpleTransmission</type>
-        <joint name="${joint}" role = "joint_1">
-            <mechanicalReduction>1.0</mechanicalReduction>
-        </joint>
-        <actuator name="${joint}_motor" role = "actuator_1"/>
-    </transmission>
-</xacro:macro>
 <!--Links-->
 <!-- World link-->
@@ -198,4 +200,35 @@
     <mimic joint = "claw_support_to_right_gripper_finger" multiplier = "-1.0"/>
 </joint>
+<!-- Sensors -->
+<!-- Camera -->
+<!-- Camera link -->
+<link name="rgb_camera">
+    <xacro:default_inertial mass="0.001"/>
+    <visual>
+        <origin xyz="-0.08 0.13 0.13" rpy="${-PI/2} 0 ${-PI/2}"/>
+        <geometry>
+            <mesh filename = "package://arduinobot_description/meshes/pi_camera.STL" scale = "0.01 0.01 0.01"/>
+        </geometry>
+    </visual>
+    <collision>
+        <origin xyz="-0.08 0.13 0.13" rpy="${-PI/2} 0 ${-PI/2}"/>
+        <geometry>
+            <mesh filename = "package://arduinobot_description/meshes/pi_camera.STL" scale = "0.01 0.01 0.01"/>
+        </geometry>
+    </collision>
+</link>
+<!-- Camera joint -->
+<joint name="rgb_camera_joint" type="fixed">
+    <parent link="base_link"/>
+    <child link="rgb_camera"/>
+    <origin xyz="0 0.45 0.2" rpy="0 -0.5 ${PI/2}"/>
+</joint>
+<!-- Camera optical link -->
+<link name="rgb_camera_optical"></link>
+<joint name="camera_optical_joint" type="fixed">
+    <parent link="rgb_camera"/>
+    <child link="rgb_camera_optical"/>
+    <origin xyz="0.0 0.0 0.0" rpy="${PI} ${PI/2} 0"/>
+</joint>
 <!-- Transmissions -->
 <xacro:default_transmission joint = "joint_1"/>
